File: Edgedancer81.kicad_pcb (KiCad board)
At the start: 2 copper layers, 340.4 x 120.7 mm, 179 parts, among them SW1 SW_Push, SW2 Rotary_Encoder_Switch, U1 ATmega32U4-AU, Y1 16MHz

Commit message: silkscreen and bugfixes
Parts:
- added G***: LOGO, random-keyboard-parts:edgedancer, F.Cu at (120.7, 186.7)
Connections:
- U1 pad 26: ROW_10 -> ROW_11
- U1 pad 27: ROW_11 -> ROW_10
Routing:
- net COL_7: track 169.3 -> 214.5 mm
- net ROW_11: track 403.1 -> 420.8 mm, vias 2 -> 0
- net Net-(USB1-Pad6): track 0.00 -> 16.3 mm
- net GND: track 235.2 -> 223.3 mm
- net +5V: track 172.8 -> 183.8 mm
- net ROW_0: track 502.4 -> 510.5 mm, vias 2 -> 4
- net ENC_B: track 26.8 -> 19.3 mm
- net Net-(D41-Pad2): track 0.00 -> 6.30 mm
- net Net-(D98-Pad2): track 0.00 -> 6.30 mm
- net Net-(D103-Pad2): track 0.00 -> 6.30 mm
- net Net-(D100-Pad2): track 0.00 -> 6.30 mm
- net ROW_10: track 496.9 -> 491.6 mm
- net ROW_2: track 429.0 -> 432.7 mm
- net Net-(C5-Pad1): track 18.5 -> 21.9 mm
- net COL_8: track 237.1 -> 234.5 mm
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- added copper zone on B.Cu, net GND
Other:
- outline, holes or cut-outs redrawn
- board text added: "Edgedancer81"
- board text added: "I will remember those who have been forgotten"
- board text added: "Life before death. Strength before weakness. Journey before destination."

Commit message: restructured keys
Parts:
- added G***: LOGO, random-keyboard-parts:edgedancer_102mm, B.Cu at (215.9, 135.9)
- MXBKSP1: footprint MX_Alps_Hybrid:MX-1U-NoLED -> MX_Alps_Hybrid:MX-2U-NoLED
- MX_ENTR1, MX_LSHFT1: footprint MX_Alps_Hybrid:MX-1U-NoLED -> MX_Alps_Hybrid:MX-2.25U-NoLED
- MX_GUI1, MX_LALT1, MX_LCTRL1, MX_RALT1, MX_RCTRL1, MX_RGUI1, MX_RMENU1: footprint MX_Alps_Hybrid:MX-1U-NoLED -> MX_Alps_Hybrid:MX-1.25U-NoLED
- MX_RSHFT1: footprint MX_Alps_Hybrid:MX-1U-NoLED -> MX_Alps_Hybrid:MX-2.75U-NoLED
- MX_SPACE1: footprint MX_Alps_Hybrid:MX-1U-NoLED -> MX_Alps_Hybrid:MX-6.25U-NoLED
- MX_SUPR1: footprint MX_Alps_Hybrid:MX-1U-NoLED -> MX_Alps_Hybrid:MX-1.75U-NoLED
- MX_TAB1, MX_\1: footprint MX_Alps_Hybrid:MX-1U-NoLED -> MX_Alps_Hybrid:MX-1.5U-NoLED
- moved MX_RALT1 13.5 mm to (231.0, 188.6)
- moved D24 12.9 mm to (45.2, 84.1)
- moved MX_ESC1 12.4 mm to (38.1, 84.1)
- moved MX1 12.1 mm to (57.1, 112.4)
- moved MX`1 12.1 mm to (38.1, 112.4)
- moved D48 12.1 mm to (121.9, 112.4)
- moved D37 12.1 mm to (83.8, 112.4)
- moved D43 12.1 mm to (102.9, 112.4)
- moved D53 12.1 mm to (141.0, 112.4)
- moved D59 12.1 mm to (160.0, 112.4)
- moved D64 12.1 mm to (179.1, 112.4)
- moved D69 12.1 mm to (198.1, 112.4)
- moved D75 12.1 mm to (217.2, 112.4)
- moved D81 12.1 mm to (236.2, 112.4)
- moved D93 12.1 mm to (274.3, 112.4)
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Connections:
- USB1 pad 6: Net-(USB1-Pad6) -> GND
Routing:
- net ROW_8: track 496.1 -> 142.7 mm
- net COL_4: track 405.6 -> 103.1 mm
- net COL_5: track 354.4 -> 54.4 mm
- net COL_1: track 507.4 -> 246.7 mm
- net COL_0: track 594.9 -> 336.2 mm
- net COL_2: track 446.0 -> 202.0 mm
- net COL_3: track 403.1 -> 166.7 mm
- net ROW_11: track 420.8 -> 210.9 mm
- net COL_6: track 224.9 -> 37.8 mm
- net ROW_10: track 491.6 -> 370.9 mm
- net COL_7: track 214.5 -> 122.4 mm
- net ROW_3: track 313.4 -> 366.3 mm
- net ROW_9: track 386.0 -> 348.3 mm
- net ROW_0: track 510.5 -> 543.3 mm
- net ROW_2: track 432.7 -> 401.0 mm
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Other:
- board size 340.4 x 120.7 mm -> 355.6 x 124.6 mm

Commit message: Created Gerbers
Parts:
- moved SW1 15.7 mm to (335.0, 119.1), turned to 90 degrees
- moved D73 13.2 mm to (238.9, 188.6)
- moved G*** 11.1 mm to (205.6, 131.8)
- moved D104 10.0 mm to (378.6, 179.4), turned to 270 degrees
- moved D57 8.41 mm to (167.5, 188.6)
- moved D79 8.41 mm to (262.7, 188.6)
- moved D85 3.67 mm to (286.5, 188.9)
- moved D91 1.11 mm to (310.4, 188.6)
Routing:
- net COL_4: track 103.1 -> 509.6 mm
- net COL_5: track 54.4 -> 430.1 mm
- net COL_0: track 336.2 -> 690.8 mm
- net COL_2: track 202.0 -> 556.2 mm
- net COL_1: track 246.7 -> 597.3 mm
- net ROW_8: track 142.7 -> 471.1 mm
- net COL_3: track 166.7 -> 489.0 mm
- net ROW_11: track 210.9 -> 458.8 mm
- net COL_6: track 37.8 -> 254.4 mm
- net COL_7: track 122.4 -> 300.8 mm
- net ROW_10: track 370.9 -> 459.6 mm
- net ROW_9: track 348.3 -> 399.4 mm
- net ROW_0: track 543.3 -> 515.7 mm
- net Net-(R3-Pad2): track 49.4 -> 29.5 mm
- net ENC_SW: track 22.9 -> 41.2 mm
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- added copper zone on F.Cu, net GND
Other:
- outline, holes or cut-outs redrawn

Commit message: fixing acute angles in traces
Parts:
- MX-1, MX0, MX1, MX2, MX3, MX4, MX5, MX6, MX7, MX8, MX9, MX=1, MX_'1, MX_,1, MX_.1, MX_/1, MX_;1, MX_A1, MX_B1, MX_C1, MX_D1, MX_DOWN1, MX_E1, MX_ESC1, MX_F1, MX_F10, MX_F11, MX_F12, MX_F13, MX_F2, MX_F3, MX_F4, MX_F5, MX_F6, MX_F7, MX_F8, MX_F9, MX_G1, MX_H1, MX_I1, MX_J1, MX_K1, MX_L1, MX_LEFT1, MX_M1, MX_N1, MX_NEXT1, MX_O1, MX_P1, MX_PLAY1, MX_PREV1, MX_Q1, MX_R1, MX_RIGHT1, MX_S1, MX_T1, MX_U1, MX_UP1, MX_V1, MX_W1, MX_X1, MX_Y1, MX_Z1, MX_[1, MX_]1, MX`1: footprint MX_Alps_Hybrid:MX-1U-NoLED -> MX_Only:MXOnly-1U-NoLED
- MXBKSP1: footprint MX_Alps_Hybrid:MX-2U-NoLED -> MX_Only:MXOnly-2U-NoLED
- MX_ENTR1, MX_LSHFT1: footprint MX_Alps_Hybrid:MX-2.25U-NoLED -> MX_Only:MXOnly-2.25U-NoLED
- MX_GUI1, MX_LALT1, MX_LCTRL1, MX_RALT1, MX_RCTRL1, MX_RGUI1, MX_RMENU1: footprint MX_Alps_Hybrid:MX-1.25U-NoLED -> MX_Only:MXOnly-1.25U-NoLED
- MX_RSHFT1: footprint MX_Alps_Hybrid:MX-2.75U-NoLED -> MX_Only:MXOnly-2.75U-NoLED
- MX_SPACE1: footprint MX_Alps_Hybrid:MX-6.25U-NoLED -> MX_Only:MXOnly-6.25U-ReversedStabilizers-NoLED
- MX_SUPR1: footprint MX_Alps_Hybrid:MX-1.75U-NoLED -> MX_Only:MXOnly-1.75U-NoLED
- MX_TAB1, MX_\1: footprint MX_Alps_Hybrid:MX-1.5U-NoLED -> MX_Only:MXOnly-1.5U-NoLED
- moved C6 5.78 mm to (319.9, 150.8)
- moved R2 2.77 mm to (321.5, 118.3)
- moved R1 2.65 mm to (319.1, 118.3)
- moved C7 2.47 mm to (322.3, 144.5)
Routing:
- net COL_2: track 556.2 -> 521.8 mm
- net COL_4: track 509.6 -> 476.8 mm
- net COL_3: track 489.0 -> 459.4 mm
- net COL_5: track 430.1 -> 402.8 mm
- net +5V: track 183.8 -> 157.6 mm, vias 6 -> 5
- net COL_6: track 254.4 -> 237.9 mm
- net COL_0: track 690.8 -> 702.2 mm
- net ROW_0: track 515.7 -> 506.3 mm
- net ROW_1: track 397.0 -> 389.4 mm
- net D+: track 43.2 -> 36.2 mm
- net COL_1: track 597.3 -> 590.4 mm
- net D-: track 43.3 -> 36.5 mm
- net ROW_7: track 425.7 -> 419.5 mm
- net COL_7: track 300.8 -> 296.3 mm
- net VCC: track 33.4 -> 29.4 mm
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
Commit message: final traces
Parts:
- moved C2 1.28 mm to (336.6, 154.8), turned to 270 degrees
- moved D24 0.79 mm to (46.0, 84.1)
- moved C1 0.78 mm to (329.4, 134.0)
- moved R3 0.70 mm to (325.4, 134.0)
Routing:
- net GND: track 212.0 -> 186.6 mm
- net ROW_6: track 516.7 -> 500.4 mm
- net ROW_9: track 399.4 -> 385.4 mm
- net ROW_5: track 447.7 -> 434.1 mm
- net +5V: track 157.6 -> 144.7 mm
- net ROW_4: track 406.6 -> 395.1 mm
- net ROW_3: track 365.5 -> 354.7 mm
- net ROW_11: track 459.7 -> 449.7 mm
- net ROW_7: track 419.5 -> 410.6 mm
- net ROW_10: track 460.4 -> 451.5 mm
- net COL_5: track 402.8 -> 394.6 mm
- net ROW_8: track 471.1 -> 463.7 mm
- net COL_4: track 476.8 -> 470.1 mm
- net ROW_2: track 402.8 -> 397.4 mm
- net COL_2: track 521.8 -> 525.4 mm
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